Commit message: Change lidar height

File: ford_fusion_2017_calibration_folder/vehicle/calibration/urdf/carma.urdf (robot description, URDF)
Before this commit: robot vehicle_platform, 9 links, 8 joints
Joints:
- joint base_link_to_ouster: origin xyz=1.35 0 1.59 rpy=0 0.0523599 0 -> xyz=1.19 0 2.03 rpy=0 0 0
- joint base_link_to_velodyne: origin xyz=1.35 0 1.59 rpy=0 0.0523599 0 -> xyz=1.19 0 2.03 rpy=0 0 0

Commit message: Updated config files

File: ford_fusion_2017_calibration_folder/vehicle/calibration/urdf/carma.urdf (robot description, URDF)
Before this commit: robot vehicle_platform, 9 links, 8 joints
Links:
- added link radar
Joints:
- added joint base_link_to_radar: type fixed, parent base_link, child radar, origin xyz=4.235 0 0.495 rpy=0 0 0
